File: PCB/FPV-Auto.brd (EAGLE design)
At the start: 65.5 x 30.7 mm, 99 parts, among them Q310 CSD25402Q3A, Q320 BSS138, U100 ATMEGA328P-AU, U110 NRF24L01+_MINI, U120 74LVC2T45DCT, U140 DRV8835, U200 RASPBERRY_PI_ZERO_W_V1.1_GPIO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, U210 MAX98357A, U300 BQ25892, U330 TPS61236P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

Commit message: pcb-update
Parts:
- R301: value ? -> 330R
- U100: value ATMEGA328P-AU -> ATMEGA328P-MU
Changed lines of the file:
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@@
 <layers>
 <layer number="1" name="Top" color="4" fill="1" visible="yes" active="yes"/>
-<layer number="2" name="GND" color="3" fill="1" visible="yes" active="yes"/>
+<layer number="2" name="GND" color="3" fill="1" visible="no" active="yes"/>
 <layer number="3" name="Route3" color="4" fill="3" visible="no" active="no"/>
 <layer number="14" name="Route14" color="1" fill="6" visible="no" active="no"/>
-<layer number="15" name="Route15" color="5" fill="1" visible="yes" active="yes"/>
-<layer number="16" name="Bottom" color="1" fill="1" visible="yes" active="yes"/>
+<layer number="15" name="Route15" color="5" fill="1" visible="no" active="yes"/>
+<layer number="16" name="Bottom" color="1" fill="1" visible="no" active="yes"/>
 <layer number="17" name="Pads" color="2" fill="1" visible="yes" active="yes"/>
 <layer number="18" name="Vias" color="2" fill="1" visible="yes" active="yes"/>
 <layer number="19" name="Unrouted" color="6" fill="1" visible="yes" active="yes"/>
 <layer number="20" name="Dimension" color="15" fill="1" visible="yes" active="yes"/>
-<layer number="21" name="tPlace" color="7" fill="1" visible="no" active="yes"/>
+<layer number="21" name="tPlace" color="7" fill="1" visible="yes" active="yes"/>
 <layer number="22" name="bPlace" color="7" fill="1" visible="no" active="yes"/>
-<layer number="23" name="tOrigins" color="15" fill="1" visible="no" active="yes"/>
+<layer number="23" name="tOrigins" color="15" fill="1" visible="yes" active="yes"/>
 <layer number="24" name="bOrigins" color="15" fill="1" visible="no" active="yes"/>
 <layer number="25" name="tNames" color="7" fill="1" visible="no" active="yes"/>
@@
 <layer number="27" name="tValues" color="7" fill="1" visible="no" active="yes"/>
 <layer number="28" name="bValues" color="7" fill="1" visible="no" active="yes"/>
-<layer number="29" name="tStop" color="7" fill="3" visible="yes" active="yes"/>
-<layer number="30" name="bStop" color="7" fill="6" visible="yes" active="yes"/>
-<layer number="31" name="tCream" color="7" fill="4" visible="yes" active="yes"/>
-<layer number="32" name="bCream" color="7" fill="5" visible="yes" active="yes"/>
+<layer number="29" name="tStop" color="7" fill="3" visible="no" active="yes"/>
+<layer number="30" name="bStop" color="7" fill="6" visible="no" active="yes"/>
+<layer number="31" name="tCream" color="7" fill="4" visible="no" active="yes"/>
+<layer number="32" name="bCream" color="7" fill="5" visible="no" active="yes"/>
 <layer number="33" name="tFinish" color="6" fill="3" visible="no" active="yes"/>
 <layer number="34" name="bFinish" color="6" fill="6" visible="no" active="yes"/>
@@
 <layer number="49" name="Reference" color="7" fill="1" visible="no" active="yes"/>
 <layer number="50" name="dxf" color="7" fill="1" visible="no" active="no"/>
-<layer number="51" name="tDocu" color="7" fill="1" visible="no" active="yes"/>
+<layer number="51" name="tDocu" color="7" fill="1" visible="yes" active="yes"/>
 <layer number="52" name="bDocu" color="7" fill="1" visible="no" active="yes"/>
 <layer number="53" name="tGND_GNDA" color="7" fill="1" visible="no" active="no"/>
@@
 <elements>
 <element name="U300" library="FPV-Auto" package="RTW(S-PWQFN-N24)_LONG" value="BQ25892" x="25.61" y="9.5" rot="R90"/>
-<element name="U100" library="FPV-Auto" package="PBS(S-PQFP-G32)" value="ATMEGA328P-AU" x="26.11" y="10" rot="MR270">
+<element name="U100" library="FPV-Auto" package="PBS(S-PQFP-G32)" value="ATMEGA328P-MU" x="26.11" y="10" rot="MR270">
 <attribute name="OC_MOUSER" value="556-ATMEGA328P-AU" x="26.11" y="10" size="1.778" layer="28" rot="MR270" display="off"/>
 </element>
@@
 <attribute name="TP_SIGNAL_NAME" value="" x="28.91" y="11.9" size="1.778" layer="27" font="vector" rot="R90" display="off"/>
 </element>
-<element name="R301" library="FPV-Auto" package="R0603" value="?" x="31.1" y="10.3" rot="R180"/>
+<element name="R301" library="FPV-Auto" package="R0603" value="330R" x="31.1" y="10.3" rot="R180"/>
 <element name="R302" library="FPV-Auto" package="R0603" value="10K" x="31.1" y="8.7" rot="R180"/>
 <element name="C304" library="FPV-Auto" package="C0805" value="10µF" x="24.21" y="14.5" rot="R270"/>
