File: PCB/FPV-Auto.sch (EAGLE design)
At the start: 97 parts, among them Q310 CSD25402Q3A, Q320 BSS138, U100 ATMEGA328P-AU, U110 NRF24L01+_MINI, U120 74LVC2T45DCT, U140 DRV8835, U200 RASPBERRY_PI_ZERO_W_V1.1_GPIO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, U210 MAX98357A, U300 BQ25892, U330 TPS61236P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

Commit message: pcb-update
Parts:
- R301: value ? -> 330R
- U100: value ATMEGA328P-AU -> ATMEGA328P-MU; device FPV-Auto:ATMEGA328P-AU -> FPV-Auto:ATMEGA328P-MU
Changed lines of the file:
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@@
 <parts>
 <part name="U300" library="FPV-Auto" deviceset="BQ25892" device=""/>
-<part name="U100" library="FPV-Auto" deviceset="ATMEGA328P" device="-AU"/>
+<part name="U100" library="FPV-Auto" deviceset="ATMEGA328P" device="-MU"/>
 <part name="U350" library="FPV-Auto" deviceset="LP5907MFX-3.3/NOPB" device=""/>
 <part name="U200" library="FPV-Auto" deviceset="RASPBERRY_PI_ZERO_W_V1.1_GPIO" device="_DUAL" value="RASPBERRY_PI_ZERO_W_V1.1_GPIO_DUAL"/>
@@
 <part name="C302" library="FPV-Auto" deviceset="C" device="0603" value="4,7µF"/>
 <part name="TP300" library="testpad" deviceset="TP" device="B1,27"/>
-<part name="R301" library="FPV-Auto" deviceset="R" device="" value="?"/>
+<part name="R301" library="FPV-Auto" deviceset="R" device="" value="330R"/>
 <part name="R302" library="FPV-Auto" deviceset="R" device="" value="10K"/>
 <part name="C304" library="FPV-Auto" deviceset="C" device="0805" value="10µF"/>
